Commit message: Added visual slam

File: description/camera.xacro (robot description, xacro)
@@ -39,5 +39,5 @@
             </camera>
             <plugin name="camera_controller" filename="libgazebo_ros_camera.so">
-                <frame_name>camera_link_optical</frame_name>
+                <frameName>camera_link_optical</frameName>
             </plugin>
         </sensor>

File: description/depth_camera.xacro (robot description, xacro)
@@ -1,10 +1,10 @@
 <?xml version="1.0"?>
 <robot xmlns:xacro="http://www.ros.org/wiki/xacro">
-    <joint name="camera_joint" type="fixed">
+    <joint name="depth_camera_joint" type="fixed">
         <parent link="chassis" />
-        <child link="camera_link" />
+        <child link="depth_camera_link" />
         <origin xyz="0.305 0 0.08" rpy="0 0 0" />
     </joint>
-    <link name="camera_link">
+    <link name="depth_camera_link">
         <visual>
             <geometry>
@@ -14,13 +14,13 @@
         </visual>
     </link>
-    <joint name="camera_optical_joint" type="fixed">
-        <parent link="camera_link" />
-        <child link="camera_link_optical" />
+    <joint name="depth_camera_optical_joint" type="fixed">
+        <parent link="depth_camera_link" />
+        <child link="depth_camera_link_optical" />
         <origin xyz="0 0 0" rpy="${-pi/2} 0 ${-pi/2}" />
     </joint>
-    <link name="camera_link_optical"></link>
+    <link name="depth_camera_link_optical"></link>
     <gazebo reference="camera_link">
         <material>Gazebo/Red</material>
-        <sensor name="camera" type="depth">
+        <sensor name="depth_camera" type="depth">
             <pose>0 0 0 0 0 0 </pose>
             <visualize>true</visualize>
@@ -39,5 +39,5 @@
             </camera>
             <plugin name="camera_controller" filename="libgazebo_ros_camera.so">
-                <frame_name>camera_link_optical</frame_name>
+                <frame_name>depth_camera_link_optical</frame_name>
                 <min_depth>0.1</min_depth>
                 <max_depth>100.0</max_depth>

File: description/robot.urdf.xacro (robot description, xacro)
@@ -3,5 +3,6 @@
     <xacro:arg name="use_ros2_control" default="true" />
     <xacro:include filename="robot_core.xacro" />
-    <xacro:include filename="lidar.xacro" />
+    <xacro:include filename="stereo_camera.xacro" />
+    <xacro:include filename="depth_camera.xacro" />
     <xacro:if value="$(arg use_ros2_control)">
         <xacro:include filename="ros2_control.xacro" />
@@ -11,5 +12,5 @@
     </xacro:unless>
     <!--
-        <xacro:include filename="camera.xacro" /
+        <xacro:include filename="lidar.xacro" />
         <xacro:include filename="depth_camera.xacro" />
     -->

File: description/robot_core.xacro (robot description, xacro)
@@ -16,4 +16,7 @@
     <material name="red">
         <color rgba="1 0 0 1"/>
+    </material>
+    <material name="green">
+        <color rgba="0.2 1 0.2 1"/>
     </material>
     <!-- BASE LINK -->

File: description/stereo_camera.xacro (robot description, xacro)
@@ -23,4 +23,17 @@
         </visual>
     </link>
+    <link name="imu_link">
+        <visual>
+            <geometry>
+                <box size="0.010 0.03 0.03" />
+            </geometry>
+            <material name="green" />
+        </visual>
+    </link>
+    <joint name="imu_joint" type="fixed">
+        <parent link="camera_link" />
+        <child link="imu_link" />
+        <origin xyz="0 0 0" rpy="0 0 0" />
+    </joint>
     <joint name="left_camera_joint" type="fixed">
         <parent link="camera_link" />
@@ -50,5 +63,5 @@
             <pose>0 0 0 0 0 0 </pose>
             <visualize>true</visualize>
-            <update_rate>30</update_rate>
+            <update_rate>60</update_rate>
             <camera>
                 <horizontal_fov>1.089</horizontal_fov>
@@ -64,5 +77,5 @@
             </camera>
             <plugin name="left_camera_controller" filename="libgazebo_ros_camera.so">
-                <frameName>left_camera_link_optical</frameName>
+                <frame_name>left_camera_link_optical</frame_name>
             </plugin>
         </sensor>
@@ -73,5 +86,5 @@
             <pose>0 0 0 0 0 0 </pose>
             <visualize>true</visualize>
-            <update_rate>30</update_rate>
+            <update_rate>60</update_rate>
             <camera>
                 <horizontal_fov>1.089</horizontal_fov>
@@ -87,7 +100,26 @@
             </camera>
             <plugin name="right_camera_controller" filename="libgazebo_ros_camera.so">
-                <frameName>right_camera_link_optical</frameName>
+                <frame_name>right_camera_link_optical</frame_name>
             </plugin>
         </sensor>
     </gazebo>
+    <gazebo reference="imu_link">
+        <gravity>true</gravity>
+        <sensor name="imu_sensor" type="imu">
+            <always_on>true</always_on>
+            <update_rate>100</update_rate>
+            <visualize>true</visualize>
+            <plugin filename="libgazebo_ros_imu_sensor.so" name="realsense_imu">
+                <topic>imu</topic>
+                <bodyName>imu_link</bodyName>
+                <updateRateHZ>10.0</updateRateHZ>
+                <gaussianNoise>0.0</gaussianNoise>
+                <xyzOffset>0 0 0</xyzOffset>
+                <rpyOffset>0 0 0</rpyOffset>
+                <frameName>imu_link</frameName>
+                <initialOrientationAsReference>false</initialOrientationAsReference>
+            </plugin>
+            <pose>0 0 0 0 0 0</pose>
+        </sensor>
+    </gazebo>
 </robot>
